File: first_test.kicad_sch (KiCad schematic)
At the start: 11 parts, among them J1 USB-C, J3 Conn_01x04, U1 STM32F103C6Ux, U2 TDN_5-0910WISM, Y1 8Mhz

Commit message: feat: add customize symbol and footprint
Signed-off-by: briq <990647625@qq.com>
Parts:
- removed C4: 1.2pf, Capacitor_SMD:C_0201_0603Metric_Pad0.64x0.40mm_HandSolder, symbol Device:C
- removed J1: USB-C, Connector_USB:USB_C_Receptacle_G-Switch_GT-USB-7025, symbol Connector:USB_C_Receptacle_PowerOnly_6P
- removed U2: TDN_5-0910WISM, Converter_DCDC:Converter_DCDC_TRACO_TDN_5-xxxxWISM_SMD, symbol Regulator_Switching:TDN_5-0910WISM
- added C4, C5: 10uf, Capacitor_SMD:C_0603_1608Metric, symbol Device:C_Polarized_Small_US
- added R2, R3: 10k, Resistor_SMD:R_0603_1608Metric, symbol Device:R
- added U2: usb type-c, first_test:usb_c_6pin, symbol first_test:usb_c_6p
- added U4: AMS1117-3.3, Package_TO_SOT_SMD:SOT-223-3_TabPin2, symbol Regulator_Linear:AMS1117-3.3
- C1, C2: value 1.2pf -> 18pf; footprint Capacitor_SMD:C_0201_0603Metric_Pad0.64x0.40mm_HandSolder -> Capacitor_SMD:C_0603_1608Metric
- C3: value 1.2pf -> 100uf; footprint Capacitor_SMD:C_0201_0603Metric_Pad0.64x0.40mm_HandSolder -> Capacitor_SMD:CP_Elec_8x10.5
- J3: footprint Connector_PinHeader_1.27mm:PinHeader_1x04_P1.27mm_Horizontal -> Connector_PinHeader_2.54mm:PinHeader_1x04_P2.54mm_Horizontal
- R1: value 2k -> 40k; footprint Resistor_SMD:R_0201_0603Metric -> Resistor_SMD:R_0603_1608Metric
- SW1: value ~ -> switch
- U1: footprint Package_DFN_QFN:QFN-48-1EP_7x7mm_P0.5mm_EP5.6x5.6mm -> Package_QFP:LQFP-48-1EP_7x7mm_P0.5mm_EP3.6x3.6mm
- Y1: footprint Crystal:Crystal_HC49-4H_Vertical -> Crystal:Crystal_SMD_HC49-SD
Connections:
- net +3.3V: now also C4.1, U4.2 (VO)
- net GND: now also C4.2, C5.2, R2.2, R3.2, U2.7 (EH), U2.A12 (GND), U2.B12 (GND), U4.1 (GND)
- new net +5V: C5.1, U2.A9 (VBUS), U2.B9 (VBUS), U4.3 (VI)
- no-connect marks 38 -> 39
